Commit message: make it compatible with ur3e model

File: rh_p12_rn_description/urdf/rh_p12_rn.xacro (robot description, xacro)
@@ -1,4 +1,4 @@
 <?xml version="1.0"?>
-<robot name="rh_p12_rn" xmlns:xacro="http://www.ros.org/wiki/xacro">
+<robot xmlns:xacro="http://www.ros.org/wiki/xacro">
   <!-- some parameters -->
   <xacro:property name="pi" value="3.141592654" />
@@ -8,9 +8,7 @@
   <xacro:include filename="$(find rh_p12_rn_description)/urdf/materials.xacro" />
   <!-- Used for fixing robot to Gazebo 'link 1' -->
-  <link name="world">
-  </link>
-  <joint name="world_fixed" type="fixed">
+  <joint name="wrist_3_link_fixed" type="fixed">
     <origin xyz="0 0 0" rpy="0 0 0"/>
-    <parent link="world"/>
+    <parent link="wrist_3_link"/>
     <child link="rh_p12_rn_base"/>
   </joint>
@@ -49,8 +47,8 @@
     <type>transmission_interface/SimpleTransmission</type>
     <joint name="rh_p12_rn">
-      <hardwareInterface>hardware_interface/EffortJointInterface</hardwareInterface>
+      <hardwareInterface>hardware_interface/PositionJointInterface</hardwareInterface>
     </joint>
     <actuator name="motor_r1">
-      <hardwareInterface>hardware_interface/EffortJointInterface</hardwareInterface>
+      <hardwareInterface>hardware_interface/PositionJointInterface</hardwareInterface>
       <mechanicalReduction>1</mechanicalReduction>
     </actuator>
@@ -90,8 +88,8 @@
     <type>transmission_interface/SimpleTransmission</type>
     <joint name="rh_r2">
-      <hardwareInterface>hardware_interface/EffortJointInterface</hardwareInterface>
+      <hardwareInterface>hardware_interface/PositionJointInterface</hardwareInterface>
     </joint>
     <actuator name="motor_r2">
-      <hardwareInterface>hardware_interface/EffortJointInterface</hardwareInterface>
+      <hardwareInterface>hardware_interface/PositionJointInterface</hardwareInterface>
       <mechanicalReduction>1</mechanicalReduction>
     </actuator>
@@ -131,8 +129,8 @@
     <type>transmission_interface/SimpleTransmission</type>
     <joint name="rh_l1">
-      <hardwareInterface>hardware_interface/EffortJointInterface</hardwareInterface>
+      <hardwareInterface>hardware_interface/PositionJointInterface</hardwareInterface>
     </joint>
     <actuator name="motor_l1">
-      <hardwareInterface>hardware_interface/EffortJointInterface</hardwareInterface>
+      <hardwareInterface>hardware_interface/PositionJointInterface</hardwareInterface>
       <mechanicalReduction>1</mechanicalReduction>
     </actuator>
@@ -172,8 +170,8 @@
     <type>transmission_interface/SimpleTransmission</type>
     <joint name="rh_l2">
-      <hardwareInterface>hardware_interface/EffortJointInterface</hardwareInterface>
+      <hardwareInterface>hardware_interface/PositionJointInterface</hardwareInterface>
     </joint>
     <actuator name="motor_l2">
-      <hardwareInterface>hardware_interface/EffortJointInterface</hardwareInterface>
+      <hardwareInterface>hardware_interface/PositionJointInterface</hardwareInterface>
       <mechanicalReduction>1</mechanicalReduction>
     </actuator>

Commit message: add gripper end effector link

File: rh_p12_rn_description/urdf/rh_p12_rn.xacro (robot description, xacro)
@@ -199,3 +199,29 @@
     </inertial>
   </link>
+  <!-- Gripper end effector joint -->
+  <joint name="rh_p12_rn_ee_joint" type="fixed">
+    <origin xyz="0.0 0.0 0.125" rpy="0 0 0"/>
+    <parent link="rh_p12_rn_base"/>
+    <child link="rh_p12_rn_ee"/>
+  </joint>
+  <!-- Gripper end effector link -->
+  <link name="rh_p12_rn_ee">
+    <visual>
+      <origin xyz="0 0 0" rpy="0 0 0"/>
+      <geometry>
+        <box size="0.01 0.01 0.01" />
+      </geometry>
+      <material name="red"/>
+     </visual>
+    <inertial>
+      <origin xyz="0 0 0" />
+      <mass value="1.0e-03" />
+      <inertia ixx="1.0e-03" ixy="0.0" ixz="0.0"
+               iyy="1.0e-03" iyz="0.0"
+               izz="1.0e-03" />
+    </inertial>
+  </link>
+  <gazebo reference="rh_p12_rn_ee">
+    <material>Gazebo/Red</material>
+  </gazebo>
 </robot>
